File: FP/FP.kicad_pcb (KiCad board)
At the start: 2 copper layers, 30 x 128.5 mm, 1 part

Commit message: why not make a front panel? lol
Parts:
- added G***: LOGO, Library:hagiwo_logo_8x8mm, F.Cu at (129.4, 154.9)
- added REF**: Thonkiconn, Library:Thonkiconn, F.Cu at (114.1, 140.4)
- added REF**: Thonkiconn, Library:Thonkiconn, F.Cu at (129.1, 140.4)
- added REF**: Thonkiconn, Library:Thonkiconn, F.Cu at (129.1, 90.4)
- added REF**: Davies1900H, Library:Davies1900H, F.Cu at (121.6, 50.4)
- added REF**: tact, Library:tact, F.Cu at (114.1, 124.8)
- added REF**: Davies1900H, Library:Davies1900H, F.Cu at (121.5, 70.4)
- added REF**: 042oled, Library:042oled, F.Cu at (129.2, 124.8)
- added REF**: Davies1900H, Library:Davies1900H, F.Cu at (114.1, 90.4)
Other:
- outline, holes or cut-outs redrawn
